File: imuwb.brd (EAGLE design)
At the start: 13 x 13.5 mm, 13 parts

Commit message: new version
Parts:
- added C4: 100nf, ipc-7351-capacitor:CAPC1005X60N
- added U$1: MIC53533.3V, bell-card:MIC5353
- added U$2: BATPADS, custom:BATPADS
- moved C3 2.62 mm to (4.25, 5.85), turned to 270 degrees
- moved R1 2.53 mm to (8.37, 11.9)
- moved C1 2.34 mm to (9.24, 11.7), turned to 270 degrees
- moved R3 1.46 mm to (3.30, 4.80), turned to 270 degrees
- moved OSC 1.44 mm to (5.88, 5.58)
- moved C2 1.04 mm to (3.07, 7.47), turned to 270 degrees
- moved MCP2210 0.79 mm to (9.58, 5.43)
- moved BME 0.77 mm to (11.0, 11.4)
- moved BMF 0.70 mm to (5.13, 10.7)
- moved AAT3681 0.60 mm to (1.79, 4.34)
- moved R2 0.45 mm to (4.33, 3.23)
Connections:
- net CSE renamed CS_ENV
- removed net CS: DWM.P$41, MCP2210.P$11
- removed net CSB: BMF.P$27, MCP2210.P$4
- removed net IRQ: BMF.P$16, DWM.P$46
- removed net RSTN: DWM.P$27
- removed net RST_MCP: BMF.P$18, MCP2210.P$1, R1.1
- removed net SUSP: BMF.P$26, MCP2210.P$3
- new net CS_ACC: BMF.P$22, MCP2210.P$2
- new net CS_DWM: DWM.P$41, MCP2210.P$12
- new net CS_GYR: BMF.P$12, MCP2210.P$3
- new net IRQ_DW: BMF.P$16, DWM.P$46, MCP2210.P$11
- new net N$4: C4.2, U$1.P$4
- new net N$5: MCP2210.P$1, R1.1
- new net VBAT: AAT3681.3, C3.1, U$1.P$1, U$1.P$3, U$2.P$2
- net +3V3: now also MCP2210.P$14, U$1.P$6; no longer AAT3681.1, AAT3681.3, BMF.P$4, C3.2
- net GND: now also C3.2, C4.1, U$1.P$2, U$1.P$7, U$2.P$1; no longer C3.1
- net RESET: now also DWM.P$27, MCP2210.P$4
- net VBUS: now also AAT3681.1; no longer MCP2210.P$14
Routing:
- net RESET: track 0.00 -> 16.8 mm, vias 0 -> 2
- net IRQ_DW: track 0.00 -> 14.3 mm, vias 0 -> 1
- net CS_GYR: track 0.00 -> 10.5 mm, vias 0 -> 2
- net +3V3: track 33.8 -> 25.0 mm, vias 2 -> 6
- net CSB: track 8.09 -> 0.00 mm
- net IRQ: track 7.78 -> 0.00 mm, vias 1 -> 0
- net MOSI: track 22.1 -> 14.9 mm, vias 1 -> 3
- net SUSP: track 6.62 -> 0.00 mm
- net GND: track 2.84 -> 8.02 mm, vias 23 -> 31
- net CS_ACC: track 0.00 -> 4.55 mm
- net MISO: track 20.3 -> 15.9 mm, vias 2 -> 3
- net N$5: track 0.00 -> 4.05 mm
- net VBUS: track 20.3 -> 16.3 mm, vias 3 -> 4
- net RST_MCP: track 3.73 -> 0.00 mm
- net N$4: track 0.00 -> 3.50 mm
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- added copper zone on layer 1, net +3V3
- added copper zone on layer 16, net VBAT
Other:
- board text added: "-"
- board text removed: "BAT"
